File: RAK11300/RAK11300_BREAKOUT.kicad_pcb (KiCad board)
At the start: 2 copper layers, 29.4 x 52 mm, 5 parts, among them J1 Conn_01x20_Male, J2 Conn_01x20_Male, J3 Conn_01x20_Male, U1 RAK11300

Commit message: pcb:(DIL_BREAKOUT_PCB RAK 11300)single gerber
Parts:
- moved REF** 2.92 mm to (63.0, 56.2)
Other:
- board text added: "1 2 3 4 5 6 7 8 9 10 11 12 13 15 16 18 19 20 21 22"
- board text added: "46 45 43 42 41 39 38 35 34 33 32 31 30 29 28 27 26 25 24 23"
Changed lines of the file:
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@@
   (general
     (thickness 1.6)
-    (drawings 6)
+    (drawings 9)
     (tracks 360)
     (zones 0)
@@
     (descr "Through hole straight pin header, 1x20, 2.54mm pitch, single row")
     (tags "Through hole pin header THT 1x20 2.54mm single row")
-    (fp_text reference J3 (at 0 -2.33) (layer F.SilkS)
+    (fp_text reference J3 (at -6.90484 -0.57) (layer F.SilkS)
       (effects (font (size 1 1) (thickness 0.15)))
     )
@@
   )
   (module Symbol:OSHW-Symbol_6.7x6mm_SilkScreen (layer F.Cu)
-    (at 61.40704 53.7718)
+    (at 62.95644 56.24576)
     (descr "Open Source Hardware Symbol")
     (tags "Logo Symbol OSHW")
@@
     (tags "LoRa LoRaWAN RAK11300")
     (attr smd)
-    (fp_text reference U1 (at -11.43 -20.32) (layer F.SilkS)
+    (fp_text reference U1 (at -7.44888 15.63144) (layer F.SilkS)
       (effects (font (size 1 1) (thickness 0.15)))
     )
@@
     (descr "Through hole straight pin header, 1x20, 2.54mm pitch, single row")
     (tags "Through hole pin header THT 1x20 2.54mm single row")
-    (fp_text reference J2 (at 0 -2.33) (layer F.SilkS)
+    (fp_text reference J2 (at -7.85988 -0.57) (layer F.SilkS)
       (effects (font (size 1 1) (thickness 0.15)))
     )
@@
     (descr "Through hole straight pin header, 1x20, 2.54mm pitch, single row")
     (tags "Through hole pin header THT 1x20 2.54mm single row")
-    (fp_text reference J1 (at 0 -2.33) (layer F.SilkS)
+    (fp_text reference J1 (at 2.96052 -0.57) (layer F.SilkS)
       (effects (font (size 1 1) (thickness 0.15)))
     )
@@
     )
   )
-  (gr_text "RAK11300 \nBREAKOUT \nV0" (at 66.51752 98.8822) (layer B.SilkS)
+  (gr_text "46\n45\n43\n42\n41\n39\n38\n35\n34\n33\n32\n31\n30\n29\n28\n27\n26\n25\n24\n23" (at 68.38696 56.8) (layer F.SilkS)
+    (effects (font (size 0.35 0.35) (thickness 0.0875)))
+  )
+  (gr_text "1\n2\n3\n4\n5\n6\n7\n8\n9\n10\n11\n12\n13\n15\n16\n18\n19\n20\n21\n22" (at 71.9582 56.8) (layer F.SilkS)
+    (effects (font (size 0.35 0.35) (thickness 0.0875)))
+  )
+  (gr_text "1\n2\n3\n4\n5\n6\n7\n8\n9\n10\n11\n12\n13\n15\n16\n18\n19\n20\n21\n22" (at 56.58104 56.8) (layer F.SilkS)
+    (effects (font (size 0.35 0.35) (thickness 0.0875)))
+  )
+  (gr_text "RAK11300 \nBREAKOUT \nV0" (at 67.21856 97.5106) (layer B.SilkS)
     (effects (font (size 1 1) (thickness 0.15)) (justify left mirror))
   )
-  (gr_text "RAK11300 \nBREAKOUT \nV0" (at 59.64936 93.40596) (layer F.SilkS)
+  (gr_text "RAK11300 \nBREAKOUT \nV0" (at 59.2836 95.0468) (layer F.SilkS)
     (effects (font (size 1 1) (thickness 0.15)) (justify left))
   )
