File: ms88sf2/ms88sf2-breakout.kicad_pcb (KiCad board)
At the start: 2 copper layers, 29.4 x 36.8 mm, 5 parts, among them J1 Conn_01x14_Male, J2 Conn_01x14_Male, J3 Conn_01x14_Male, U1 MS88SF2

Commit message: MS88SF2 routed
Parts:
- moved U1 4.45 mm to (63.4, 65.0)
- moved REF** 2.57 mm to (63.3, 56.7)
Connections:
- J2 pad 1: /ICPIN32 -> /ICPIN28
- J2 pad 10: /ICPIN21 -> /ICPIN19
- J2 pad 11: /ICPIN20 -> /ICPIN18
- J2 pad 12: /ICPIN19 -> /ICPIN17
- J2 pad 2: /ICPIN31 -> /ICPIN27
- J2 pad 3: /ICPIN30 -> /ICPIN26
- J2 pad 4: /ICPIN29 -> /ICPIN25
- J2 pad 5: /ICPIN27 -> /ICPIN24
- J2 pad 6: /ICPIN26 -> /ICPIN23
- J2 pad 7: /ICPIN25 -> /ICPIN22
- J2 pad 8: /ICPIN24 -> /ICPIN21
- J2 pad 9: /ICPIN22 -> /ICPIN20
- U1 pad 1: Net-(U1-Pad1) -> /ICPIN01
- U1 pad 10: Net-(U1-Pad10) -> /ICPIN10
- U1 pad 11: Net-(U1-Pad11) -> /ICPIN11
- U1 pad 12: Net-(U1-Pad12) -> /ICPIN12
- U1 pad 13: Net-(U1-Pad13) -> /ICPIN13
- U1 pad 14: Net-(U1-Pad14) -> /ICPIN14
- U1 pad 15: Net-(U1-Pad15) -> /ICPIN15
- U1 pad 16: Net-(U1-Pad16) -> /ICPIN16
- U1 pad 17: Net-(U1-Pad17) -> /ICPIN17
- U1 pad 18: Net-(U1-Pad18) -> /ICPIN18
- U1 pad 19: Net-(U1-Pad19) -> /ICPIN19
- U1 pad 2: Net-(U1-Pad2) -> /ICPIN02
- U1 pad 20: Net-(U1-Pad20) -> /ICPIN20
- U1 pad 21: Net-(U1-Pad21) -> /ICPIN21
- U1 pad 22: Net-(U1-Pad22) -> /ICPIN22
- U1 pad 23: Net-(U1-Pad23) -> /ICPIN23
- U1 pad 24: Net-(U1-Pad24) -> /ICPIN24
- U1 pad 25: Net-(U1-Pad25) -> /ICPIN25
- U1 pad 26: Net-(U1-Pad26) -> /ICPIN26
- U1 pad 27: Net-(U1-Pad27) -> /ICPIN27
- U1 pad 3: Net-(U1-Pad3) -> /ICPIN03
- U1 pad 4: Net-(U1-Pad4) -> /ICPIN04
- U1 pad 5: Net-(U1-Pad5) -> /ICPIN05
- U1 pad 6: Net-(U1-Pad6) -> /ICPIN06
- U1 pad 7: Net-(U1-Pad7) -> /ICPIN07
- U1 pad 8: Net-(U1-Pad8) -> /ICPIN08
- U1 pad 9: Net-(U1-Pad9) -> /ICPIN09
Routing:
- net /ICPIN03: track 0.00 -> 43.5 mm, vias 0 -> 1
- net /ICPIN02: track 0.00 -> 39.0 mm
- net /ICPIN14: track 0.00 -> 38.2 mm
- net /ICPIN01: track 0.00 -> 37.6 mm
- net /ICPIN13: track 0.00 -> 37.4 mm
- net /ICPIN12: track 0.00 -> 35.9 mm, vias 0 -> 1
- net /ICPIN11: track 0.00 -> 34.9 mm, vias 0 -> 1
- net /ICPIN04: track 0.00 -> 33.7 mm, vias 0 -> 1
- net /ICPIN05: track 0.00 -> 32.6 mm
- net /ICPIN10: track 0.00 -> 32.6 mm
- net /ICPIN09: track 0.00 -> 31.4 mm
- net /ICPIN06: track 0.00 -> 31.1 mm
- net /ICPIN08: track 0.00 -> 30.4 mm
- net /ICPIN07: track 0.00 -> 29.7 mm
- net /ICPIN16: track 0.00 -> 21.0 mm
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Other:
- board text added: "1 2 3 4 5"
- board text added: "23 22 21 20 19 18 17 16 15"
- board text added: "28 27 26 25 24"
- board text added: "6 7 8 9 10 11 12 13 14"
- board text removed: "1 2 3 4 5 6 7 8 9 10 11 12 13 14"
- board text removed: "28 27 26 25 24 23 22 21 20 19 18 17 16 15"
