File: ms88sf2/ms88sf2-breakout.sch (KiCad schematic (older format))
At the start: 4 parts, among them J1 Conn_01x14_Male, J2 Conn_01x14_Male, J3 Conn_01x14_Male, U1 MS88SF2

Commit message: MS88SF2 routed
Connections:
- net labels added: ICPIN17, ICPIN18, ICPIN23, ICPIN28
- net labels removed: ICPIN29, ICPIN30, ICPIN31, ICPIN32
- wire segments 73 -> 70
Changed lines of the file:
@@
 Wire Wire Line
 	3050 2550 3200 2550
-Wire Wire Line
-	3750 5400 4150 5400
 Text Label 6700 3500 0    50   ~ 0
 ICPIN05
-Wire Wire Line
-	3750 5500 4150 5500
 Text Label 3200 2650 0    50   ~ 0
 ICPIN05
@@
 Text Label 6700 3400 0    50   ~ 0
 ICPIN07
-Wire Wire Line
-	3750 4500 4150 4500
 Text Label 3200 2850 0    50   ~ 0
 ICPIN07
@@
 Text Label 6700 2400 0    50   ~ 0
 ICPIN09
-Wire Wire Line
-	3750 4800 4150 4800
 Text Label 3200 3050 0    50   ~ 0
 ICPIN09
@@
 Text Label 6700 2500 0    50   ~ 0
 ICPIN10
-Wire Wire Line
-	3750 4900 4150 4900
 Text Label 3200 3150 0    50   ~ 0
 ICPIN10
@@
 Wire Wire Line
 	3050 3550 3200 3550
-Text Label 3750 5000 0    50   ~ 0
+Text Label 4100 2900 0    50   ~ 0
 ICPIN16
-Wire Wire Line
-	3750 5000 4150 5000
 Text Label 7550 2950 0    50   ~ 0
-ICPIN24
+ICPIN21
 Text Label 7550 2850 0    50   ~ 0
-ICPIN25
+ICPIN22
 Text Label 7550 2750 0    50   ~ 0
-ICPIN26
-Text Label 4750 5150 0    50   ~ 0
+ICPIN23
+Text Label 4100 2600 0    50   ~ 0
 ICPIN26
 Text Label 7550 2650 0    50   ~ 0
+ICPIN24
+Text Label 6700 2600 0    50   ~ 0
+ICPIN27
+Text Label 7550 2550 0    50   ~ 0
+ICPIN25
+Text Label 6700 3300 0    50   ~ 0
+ICPIN23
+Text Label 7550 2450 0    50   ~ 0
+ICPIN26
+Text Label 7550 2350 0    50   ~ 0
 ICPIN27
 Text Label 6700 2900 0    50   ~ 0
-ICPIN27
-Text Label 7550 2550 0    50   ~ 0
-ICPIN29
-Text Label 4800 5000 0    50   ~ 0
-ICPIN29
-Text Label 7550 2450 0    50   ~ 0
-ICPIN30
-Text Label 7550 2350 0    50   ~ 0
-ICPIN31
-Text Label 6700 3300 0    50   ~ 0
-ICPIN31
+ICPIN18
 Text Label 7550 2250 0    50   ~ 0
-ICPIN32
-Text Label 6700 3200 0    50   ~ 0
-ICPIN32
+ICPIN28
+Text Label 4100 2800 0    50   ~ 0
+ICPIN17
 $Comp
 L Connector:Conn_01x14_Male J1
@@
 Text Label 6700 2300 0    50   ~ 0
 ICPIN08
-Wire Wire Line
-	3750 4600 4150 4600
 Text Label 4100 3300 0    50   ~ 0
 ICPIN11
@@
 Text Label 5550 4200 1    50   ~ 0
 ICPIN13
-Wire Wire Line
-	4150 5100 3750 5100
 Text Label 5450 1700 1    50   ~ 0
 ICPIN14
 Wire Wire Line
-	4150 5200 3750 5200
-Wire Wire Line
-	6550 3200 6700 3200
-Wire Wire Line
 	7550 2250 8000 2250
 Wire Wire Line
-	6550 3300 6700 3300
-Wire Wire Line
 	7550 2350 8000 2350
-Text Label 4700 4750 0    50   ~ 0
-ICPIN30
+Text Label 6700 2700 0    50   ~ 0
+ICPIN28
 Wire Wire Line
 	7550 2450 8000 2450
@@
 	7550 2550 8000 2550
 Wire Wire Line
-	6550 2900 6700 2900
-Wire Wire Line
 	7550 2650 8000 2650
 Wire Wire Line
 	7550 2750 8000 2750
-Text Label 4700 5350 0    50   ~ 0
+Text Label 4100 2500 0    50   ~ 0
 ICPIN25
 Wire Wire Line
 	7550 2850 8000 2850
-Text Label 5500 5100 1    50   ~ 0
+Text Label 4100 3200 0    50   ~ 0
 ICPIN24
 Wire Wire Line
 	7550 2950 8000 2950
-Text Label 3750 4300 0    50   ~ 0
+Text Label 6700 3200 0    50   ~ 0
 ICPIN22
-Wire Wire Line
-	3750 4300 4150 4300
 Text Label 7550 3050 0    50   ~ 0
-ICPIN22
+ICPIN20
 Wire Wire Line
 	7550 3050 8000 3050
-Text Label 3750 4400 0    50   ~ 0
+Text Label 6700 3100 0    50   ~ 0
 ICPIN21
-Wire Wire Line
-	3750 4400 4150 4400
 Text Label 7550 3150 0    50   ~ 0
-ICPIN21
+ICPIN19
 Wire Wire Line
 	7550 3150 8000 3150
-Text Label 6700 2700 0    50   ~ 0
+Text Label 4100 2400 0    50   ~ 0
 ICPIN20
-Wire Wire Line
-	6550 2700 6700 2700
 Text Label 7550 3250 0    50   ~ 0
-ICPIN20
+ICPIN18
 Wire Wire Line
 	7550 3250 8000 3250
-Text Label 6700 2600 0    50   ~ 0
+Text Label 6700 3000 0    50   ~ 0
 ICPIN19
-Wire Wire Line
-	6550 2600 6700 2600
 Text Label 7550 3350 0    50   ~ 0
-ICPIN19
+ICPIN17
 Wire Wire Line
 	7550 3350 8000 3350
@@
 Wire Wire Line
 	7550 3450 8000 3450
-Text Label 3750 5300 0    50   ~ 0
+Text Label 5550 1700 1    50   ~ 0
 ICPIN15
-Wire Wire Line
-	3750 5300 4150 5300
 Text Label 7550 3550 0    50   ~ 0
 ICPIN15
@@
 Wire Wire Line
 	5450 1700 5450 2000
+Wire Wire Line
+	5550 2000 5550 1700
+Wire Wire Line
+	4100 2900 4750 2900
+Wire Wire Line
+	4100 2800 4750 2800
+Wire Wire Line
+	6150 2900 6700 2900
+Wire Wire Line
+	6150 3000 6700 3000
+Wire Wire Line
+	4100 2400 4750 2400
+Wire Wire Line
+	6150 3100 6700 3100
+Wire Wire Line
+	6150 3200 6700 3200
+Wire Wire Line
+	6150 3300 6700 3300
+Wire Wire Line
+	4100 3200 4750 3200
+Wire Wire Line
+	4750 2500 4100 2500
+Wire Wire Line
+	4750 2600 4100 2600
+Wire Wire Line
+	6150 2600 6700 2600
+Wire Wire Line
+	6150 2700 6700 2700
 $EndSCHEMATC
